Commit message: updated gem description

File: src/vehicle_drivers/gem_visualization/gem_description/urdf/e4/gem_e4.urdf (robot description, URDF)
Before this commit: robot gem_e4, 31 links, 30 joints
Links:
- link base_link: geometry collision mesh filename=package://gem_description/meshes/e4/base_link.STL; visual mesh filename=package://gem_description/meshes/e4/base_link.STL
- link front_camera_link: geometry collision mesh filename=package://gem_description/meshes/e4/front_camera_link.STL; visual mesh filename=package://gem_description/meshes/e4/front_camera_link.STL
- link front_lidar_link: geometry collision mesh filename=package://gem_description/meshes/e4/front_lidar_link.STL; visual mesh filename=package://gem_description/meshes/e4/front_lidar_link.STL
- link front_rack_link: geometry collision mesh filename=package://gem_description/meshes/e4/front_rack_link.STL; visual mesh filename=package://gem_description/meshes/e4/front_rack_link.STL
- link front_radar_link: geometry collision mesh filename=package://gem_description/meshes/e4/front_radar_link.STL; visual mesh filename=package://gem_description/meshes/e4/front_radar_link.STL
- link gps_antenna_aux_link: geometry collision mesh filename=package://gem_description/meshes/e4/gps_antenna_aux_link.STL; visual mesh filename=package://gem_description/meshes/e4/gps_antenna_aux_link.STL
- link gps_antenna_main_link: geometry collision mesh filename=package://gem_description/meshes/e4/gps_antenna_main_link.S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; visual mesh filename=package://gem_description/meshes/e4/gps_antenna_main_link.S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
- link headlight_fl_link: geometry collision mesh filename=package://gem_description/meshes/e4/headlight_fl_link.STL; visual mesh filename=package://gem_description/meshes/e4/headlight_fl_link.STL
- link headlight_fr_link: geometry collision mesh filename=package://gem_description/meshes/e4/headlight_fr_link.STL; visual mesh filename=package://gem_description/meshes/e4/headlight_fr_link.STL
- link i_logo_fl_link: geometry collision mesh filename=package://gem_description/meshes/e4/i_logo_link.STL; visual mesh filename=package://gem_description/meshes/e4/i_logo_link.STL
- link i_logo_fr_link: geometry collision mesh filename=package://gem_description/meshes/e4/i_logo_link.STL; visual mesh filename=package://gem_description/meshes/e4/i_logo_link.STL
- link i_logo_rl_link: geometry collision mesh filename=package://gem_description/meshes/e4/i_logo_link.STL; visual mesh filename=package://gem_description/meshes/e4/i_logo_link.STL
- link i_logo_rr_link: geometry collision mesh filename=package://gem_description/meshes/e4/i_logo_link.STL; visual mesh filename=package://gem_description/meshes/e4/i_logo_link.STL
- link imu_link: geometry collision mesh filename=package://gem_description/meshes/e4/imu_link.STL; visual mesh filename=package://gem_description/meshes/e4/imu_link.STL
- link lightbar_link: geometry collision mesh filename=package://gem_description/meshes/e4/lightbar_link.STL; visual mesh filename=package://gem_description/meshes/e4/lightbar_link.STL
- link rear_rack_link: geometry collision mesh filename=package://gem_description/meshes/e4/rear_rack_link.STL; visual mesh filename=package://gem_description/meshes/e4/rear_rack_link.STL
- link stoplight_rl_link: geometry collision mesh filename=package://gem_description/meshes/e4/stoplight_rl_link.STL; visual mesh filename=package://gem_description/meshes/e4/stoplight_rl_link.STL
- link stoplight_rr_link: geometry collision mesh filename=package://gem_description/meshes/e4/stoplight_rr_link.STL; visual mesh filename=package://gem_description/meshes/e4/stoplight_rr_link.STL
- link taillight_rl_link: geometry collision mesh filename=package://gem_description/meshes/e4/taillight_rl_link.STL; visual mesh filename=package://gem_description/meshes/e4/taillight_rl_link.STL
- link taillight_rr_link: geometry collision mesh filename=package://gem_description/meshes/e4/taillight_rr_link.STL; visual mesh filename=package://gem_description/meshes/e4/taillight_rr_link.STL
- link top_lidar_link: geometry collision mesh filename=package://gem_description/meshes/e4/top_lidar_link.STL; visual mesh filename=package://gem_description/meshes/e4/top_lidar_link.STL
- link top_rack_link: geometry collision mesh filename=package://gem_description/meshes/e4/top_rack_link.STL; visual mesh filename=package://gem_description/meshes/e4/top_rack_link.STL
- link turnlight_fl_link: geometry collision mesh filename=package://gem_description/meshes/e4/turnlight_fl_link.STL; visual mesh filename=package://gem_description/meshes/e4/turnlight_fl_link.STL
- link turnlight_fr_link: geometry collision mesh filename=package://gem_description/meshes/e4/turnlight_fr_link.STL; visual mesh filename=package://gem_description/meshes/e4/turnlight_fr_link.STL
- link wheel_link_fl: geometry collision sphere radius=0.295; visual mesh filename=package://gem_description/meshes/e4/wheel_link_fl.STL
- link wheel_link_fr: geometry collision sphere radius=0.295; visual mesh filename=package://gem_description/meshes/e4/wheel_link_fr.STL
- link wheel_link_rl: geometry collision sphere radius=0.295; visual mesh filename=package://gem_description/meshes/e4/wheel_link_rl.STL
- link wheel_link_rr: geometry collision sphere radius=0.295; visual mesh filename=package://gem_description/meshes/e4/wheel_link_rr.STL
