Commit message: tested sensors_init on e4 ouster causing issues

File: src/vehicle_drivers/gem_visualization/gem_description/urdf/e4/gem_e4.urdf.xacro (robot description, xacro)
@@ -791,4 +791,11 @@
     </collision>
   </link>
+<link name="vsm"/>
+<!-- Fixed joint connecting imu_link to vsm -->
+<joint name="imu_to_vsm_joint" type="fixed">
+  <parent link="imu_link" />
+  <child link="vsm" />
+  <origin xyz="0 0 0" rpy="0 0 0" />
+</joint>
   <gazebo reference="imu_link">
     <material>Gazebo/White</material>
