Commit message: lidar updated in  gem_description

File: src/vehicle_drivers/gem_visualization/gem_description/urdf/e2/gem_e2.urdf.xacro (robot description, xacro)
@@ -10,4 +10,5 @@
   <xacro:include filename="$(find gem_description)/urdf/materials.xacro" />
   <xacro:include filename="$(find gem_description)/urdf/macros.xacro" />
+  <xacro:include filename="$(find gem_description)/urdf/ouster/OS1-64.urdf.xacro" />
   <!-- *************************** Base link below *************************** -->
   <link name="base_footprint">
@@ -1020,4 +1021,7 @@
   <xacro:steering_hinge_transmission name="right_steering_hinge" />
   <!-- *********************************************** Sensors ************************************************ -->
+ <xacro:OS1_64 parent="top_rack_link" name="ouster" topic_points="/ouster/points" topic_imu ="/ouster/imu" hz="10" lasers="64" samples="512" min_range="0.9" max_range="75.0" noise="0.008" min_angle="-${M_PI}" max_angle="${M_PI}" lidar_link="os_lidar" imu_link="os_imu" vfov_min="-.26" vfov_max=".26" >
+    <origin xyz="0.02 0.115 -0.6575" rpy="1.5708 0 3.1416" />
+  </xacro:OS1_64>
   <!-- ************************* Front Camera ************************* -->
   <link name="front_single_camera_link">

File: src/vehicle_drivers/gem_visualization/gem_description/urdf/e4/gem_e4.urdf.xacro (robot description, xacro)
@@ -12,5 +12,5 @@
   <xacro:include filename="$(find gem_description)/urdf/materials.xacro" />
   <xacro:include filename="$(find gem_description)/urdf/macros.xacro" />
-  <!-- <xacro:include filename="$(find velodyne_description)/urdf/OS1.urdf.xacro" /> -->
+  <xacro:include filename="$(find gem_description)/urdf/ouster/OS1-64.urdf.xacro" />
   <link name="base_footprint">
   </link>
@@ -971,7 +971,7 @@
   <xacro:steering_hinge_transmission name="right_steering_hinge" />
   <!-- *********************************************** Sensors ************************************************ -->
-  <!-- <xacro:OS1 parent="top_rack_link" name="ouster" topic="/ouster/points" hz="10" samples="440" gpu="true" lasers="128" min_range="0.5" max_range="200.0" min_angle="-${M_PI}" max_angle="${M_PI}">
+  <xacro:OS1_64 parent="top_rack_link" name="ouster" topic_points="/ouster/points" topic_imu ="/ouster/imu" hz="10" lasers="64" samples="512" min_range="0.9" max_range="75.0" noise="0.008" min_angle="-${M_PI}" max_angle="${M_PI}" lidar_link="os_lidar" imu_link="os_imu" vfov_min="-.26" vfov_max=".26" >
     <origin xyz="0.02 0.42 0" rpy="1.5708 0 3.1416" />
-  </xacro:OS1> -->
+  </xacro:OS1_64>
   <!-- ************************* Front Camera ************************* -->
   <link name="front_single_camera_link">

Commit message: sensors tested on e2

File: src/vehicle_drivers/gem_visualization/gem_description/urdf/e2/gem_e2.urdf.xacro (robot description, xacro)
@@ -1109,7 +1109,13 @@
   </link>
   <joint name="IMU_joint" type="fixed">
-    <origin xyz="-0.246 0 0.05" rpy="0 0 -1.5708"/>
+    <origin xyz="-0.05 -0.4 0.05" rpy="0 0 0"/>
     <parent link="base_link"/>
     <child link="IMU_link"/>
+  </joint>
+    <link name="vsm"/>
+  <joint name="velocity_sensor_joint" type="fixed">
+    <origin xyz="0.0 0 0.0" rpy="0 0 0"/>
+    <parent link="IMU_link"/>
+    <child link="vsm"/>
   </joint>
   <!-- GPS -->

File: src/vehicle_drivers/gem_visualization/gem_description/urdf/e4/gem_e4.urdf.xacro (robot description, xacro)
@@ -791,11 +791,4 @@
     </collision>
   </link>
-<link name="vsm"/>
-<!-- Fixed joint connecting imu_link to vsm -->
-<joint name="imu_to_vsm_joint" type="fixed">
-  <parent link="imu_link" />
-  <child link="vsm" />
-  <origin xyz="0 0 0" rpy="0 0 0" />
-</joint>
   <gazebo reference="imu_link">
     <material>Gazebo/White</material>

Commit message: gnss_control tested on e4

File: src/vehicle_drivers/gem_visualization/gem_description/urdf/e2/gem_e2.urdf.xacro (robot description, xacro)
@@ -1113,5 +1113,5 @@
     <child link="IMU_link"/>
   </joint>
-    <link name="vsm"/>
+  <link name="vsm"/>
   <joint name="velocity_sensor_joint" type="fixed">
     <origin xyz="0.0 0 0.0" rpy="0 0 0"/>

File: src/vehicle_drivers/gem_visualization/gem_description/urdf/e4/gem_e4.urdf.xacro (robot description, xacro)
@@ -800,4 +800,10 @@
     <axis xyz="0 0 0" />
   </joint>
+  <link name="vsm"/>
+  <joint name="velocity_sensor_joint" type="fixed">
+    <origin xyz="0.0 0 0.0" rpy="0 0 0"/>
+    <parent link="imu_link"/>
+    <child link="vsm"/>
+  </joint>
   <!-- *********************************** Front Left Wheel *********************************** -->
   <link name="left_steering_hinge_link">
